Commit message: Fix TF + dynamic obstacle overlay for LiDAR
Restore full TF chain and make obstacle overlay follow SLAM map geometry. Adds a fixed base_footprint->base_link joint in agv.urdf.xacro so scans (frame: laser) map to base_footprint. package.xml gains runtime/launch deps plus rplidar_ros and slam_toolbox exec_deps. map_manager_node.py removed the hardcoded 800×800 grid and now validates /map geometry, allocates a live overlay matching map width/height/resolution/origin, converts world→cell using that geometry, and publishes obstacle_layer with the same map info. Includes LIDAR_ONLY_RECOVERY_REPORT.md with diagnosis and Pi-side verification steps.

File: services/robot/src/my_robot_controller/urdf/agv.urdf.xacro (robot description, xacro)
@@ -3,5 +3,5 @@
   AGV robot description — minimal URDF for TF tree.
   Frame chain:
-    base_link → laser (LiDAR mount, ~25 cm above base, 5 cm forward)
+    base_footprint → base_link → laser (LiDAR mount, ~25 cm above base, 5 cm forward)
     base_link → base_imu (BNO055 mount, centered on chassis)
   Geometry is a 30 cm square mecanum chassis. Tune dimensions here when
@@ -10,4 +10,11 @@
 -->
 <robot name="agv" xmlns:xacro="http://ros.org/wiki/xacro">
+  <!-- Ground-projected base frame published below the physical chassis. -->
+  <link name="base_footprint"/>
+  <joint name="base_footprint_to_base_link" type="fixed">
+    <parent link="base_footprint"/>
+    <child link="base_link"/>
+    <origin xyz="0 0 0" rpy="0 0 0"/>
+  </joint>
   <!-- Base chassis (visual + collision) -->
   <link name="base_link">
